Commit message: support: add 'flange' frame.
Similar to 'tool0', but without the orientation change (to make Z+
parallel to X+).

The 'flange' frame is intended as attachment point for EEFs, while 'tool0'
is meant to be a immutable frame that always encodes an "all-zeros tool
centre point" configuration.

Both 'tool0' and 'flange' should not be changed.

File: fanuc_lrmate200ic_support/urdf/lrmate200ic5f_macro.xacro (robot description, xacro)
@@ -93,4 +93,5 @@
       </collision>
     </link>
+    <link name="${prefix}flange" />
     <link name="${prefix}tool0" />
     <joint name="${prefix}joint_1" type="revolute">
@@ -129,7 +130,12 @@
       <limit effort="0" lower="-6.285" upper="6.285" velocity="20.94395" />
     </joint>
-    <joint name="${prefix}joint_5-tool0" type="fixed">
+    <joint name="${prefix}joint_5-flange" type="fixed">
+      <origin xyz="0 0 0" rpy="0 0 0" />
+      <parent link="${prefix}link_5" />
+      <child link="${prefix}flange" />
+    </joint>
+    <joint name="${prefix}flange-tool0" type="fixed">
       <origin xyz="0 0 0" rpy="${pi} ${-pi/2.0} 0" />
-      <parent link="${prefix}link_5" />
+      <parent link="${prefix}flange" />
       <child link="${prefix}tool0" />
     </joint>

File: fanuc_lrmate200ic_support/urdf/lrmate200ic5h_macro.xacro (robot description, xacro)
@@ -93,4 +93,5 @@
       </collision>
     </link>
+    <link name="${prefix}flange" />
     <link name="${prefix}tool0" />
     <joint name="${prefix}joint_1" type="revolute">
@@ -129,7 +130,12 @@
       <limit effort="0" lower="-6.285" upper="6.285" velocity="12.5664" />
     </joint>
-    <joint name="${prefix}joint_5-tool0" type="fixed">
+    <joint name="${prefix}joint_5-flange" type="fixed">
+      <origin xyz="0 0 0" rpy="0 0 0" />
+      <parent link="${prefix}link_5" />
+      <child link="${prefix}flange" />
+    </joint>
+    <joint name="${prefix}flange-tool0" type="fixed">
       <origin xyz="0 0 0" rpy="${pi} ${-pi/2.0} 0" />
-      <parent link="${prefix}link_5" />
+      <parent link="${prefix}flange" />
       <child link="${prefix}tool0" />
     </joint>

File: fanuc_lrmate200ic_support/urdf/lrmate200ic5hs_macro.xacro (robot description, xacro)
@@ -93,4 +93,5 @@
       </collision>
     </link>
+    <link name="${prefix}flange" />
     <link name="${prefix}tool0" />
     <joint name="${prefix}joint_1" type="revolute">
@@ -129,7 +130,12 @@
       <limit effort="0" lower="-6.285" upper="6.285" velocity="20.94395" />
     </joint>
-    <joint name="${prefix}joint_5-tool0" type="fixed">
+    <joint name="${prefix}joint_5-flange" type="fixed">
+      <origin xyz="0 0 0" rpy="0 0 0" />
+      <parent link="${prefix}link_5" />
+      <child link="${prefix}flange" />
+    </joint>
+    <joint name="${prefix}flange-tool0" type="fixed">
       <origin xyz="0 0 0" rpy="${pi} ${-pi/2.0} 0" />
-      <parent link="${prefix}link_5" />
+      <parent link="${prefix}flange" />
       <child link="${prefix}tool0" />
     </joint>

File: fanuc_lrmate200ic_support/urdf/lrmate200ic5l_macro.xacro (robot description, xacro)
@@ -108,4 +108,5 @@
       </collision>
     </link>
+    <link name="${prefix}flange" />
     <link name="${prefix}tool0" />
     <joint name="${prefix}joint_1" type="revolute">
@@ -151,7 +152,12 @@
       <limit effort="0" lower="-6.2832" upper="6.2832" velocity="12.5664" />
     </joint>
-    <joint name="${prefix}joint_6-tool0" type="fixed">
+    <joint name="${prefix}joint_6-flange" type="fixed">
+      <origin xyz="0 0 0" rpy="0 0 0" />
+      <parent link="${prefix}link_6" />
+      <child link="${prefix}flange" />
+    </joint>
+    <joint name="${prefix}flange-tool0" type="fixed">
       <origin xyz="0 0 0" rpy="${pi} ${-pi/2.0} 0" />
-      <parent link="${prefix}link_6" />
+      <parent link="${prefix}flange" />
       <child link="${prefix}tool0" />
     </joint>

File: fanuc_lrmate200ic_support/urdf/lrmate200ic_macro.xacro (robot description, xacro)
@@ -108,4 +108,5 @@
       </collision>
     </link>
+    <link name="${prefix}flange" />
     <link name="${prefix}tool0" />
     <joint name="${prefix}joint_1" type="revolute">
@@ -151,7 +152,12 @@
       <limit effort="0" lower="-6.2832" upper="6.2832" velocity="12.5664" />
     </joint>
-    <joint name="${prefix}joint_6-tool0" type="fixed">
+    <joint name="${prefix}joint_6-flange" type="fixed">
+      <origin xyz="0 0 0" rpy="0 0 0" />
+      <parent link="${prefix}link_6" />
+      <child link="${prefix}flange" />
+    </joint>
+    <joint name="${prefix}flange-tool0" type="fixed">
       <origin xyz="0 0 0" rpy="${pi} ${-pi/2.0} 0" />
-      <parent link="${prefix}link_6" />
+      <parent link="${prefix}flange" />
       <child link="${prefix}tool0" />
     </joint>

File: fanuc_m10ia_support/urdf/m10ia7l_macro.xacro (robot description, xacro)
@@ -109,5 +109,6 @@
       </collision>
     </link>
-    <link name="${prefix}tool0"/>
+    <link name="${prefix}flange" />
+    <link name="${prefix}tool0" />
     <!-- joints -->
     <joint name="${prefix}joint_1" type="revolute">
@@ -153,8 +154,13 @@
       <limit lower="-6.28" upper="6.28" effort="0" velocity="11.00"/>
     </joint>
-    <joint name="${prefix}joint_6-tool0" type="fixed">
+    <joint name="${prefix}joint_6-flange" type="fixed">
+      <origin xyz="0 0 0" rpy="0 0 0" />
+      <parent link="${prefix}link_6" />
+      <child link="${prefix}flange" />
+    </joint>
+    <joint name="${prefix}flange-tool0" type="fixed">
       <origin xyz="0 0 0" rpy="${pi} ${-pi/2.0} 0" />
-      <parent link="${prefix}link_6"/>
-      <child link="${prefix}tool0"/>
+      <parent link="${prefix}flange" />
+      <child link="${prefix}tool0" />
     </joint>
     <!-- ROS base_link to Fanuc World Coordinates transform -->

File: fanuc_m10ia_support/urdf/m10ia_macro.xacro (robot description, xacro)
@@ -109,5 +109,6 @@
       </collision>
     </link>
-    <link name="${prefix}tool0"/>
+    <link name="${prefix}flange" />
+    <link name="${prefix}tool0" />
     <!-- joints -->
     <joint name="${prefix}joint_1" type="revolute">
@@ -153,8 +154,13 @@
       <limit lower="-6.28" upper="6.28" effort="0" velocity="10.47"/>
     </joint>
-    <joint name="${prefix}joint_6-tool0" type="fixed">
+    <joint name="${prefix}joint_6-flange" type="fixed">
+      <origin xyz="0 0 0" rpy="0 0 0" />
+      <parent link="${prefix}link_6" />
+      <child link="${prefix}flange" />
+    </joint>
+    <joint name="${prefix}flange-tool0" type="fixed">
       <origin xyz="0 0 0" rpy="${pi} ${-pi/2.0} 0" />
-      <parent link="${prefix}link_6"/>
-      <child link="${prefix}tool0"/>
+      <parent link="${prefix}flange" />
+      <child link="${prefix}tool0" />
     </joint>
     <!-- ROS base_link to Fanuc World Coordinates transform -->

File: fanuc_m16ib_support/urdf/m16ib20_macro.xacro (robot description, xacro)
@@ -109,5 +109,6 @@
       </collision>
     </link>
-    <link name="${prefix}tool0"/>
+    <link name="${prefix}flange" />
+    <link name="${prefix}tool0" />
     <!-- joints -->
     <joint name="${prefix}joint_1" type="revolute">
@@ -153,8 +154,13 @@
       <limit effort="0" lower="-7.8540" upper="7.8540" velocity="9.0757" />
     </joint>
-    <joint name="${prefix}joint_6-tool0" type="fixed">
+    <joint name="${prefix}joint_6-flange" type="fixed">
+      <origin xyz="0 0 0" rpy="0 0 0" />
+      <parent link="${prefix}link_6" />
+      <child link="${prefix}flange" />
+    </joint>
+    <joint name="${prefix}flange-tool0" type="fixed">
       <origin xyz="0 0 0" rpy="${pi} ${-pi/2.0} 0" />
-      <parent link="${prefix}link_6"/>
-      <child link="${prefix}tool0"/>
+      <parent link="${prefix}flange" />
+      <child link="${prefix}tool0" />
     </joint>
     <!-- ROS base_link to Fanuc World Coordinates transform -->

File: fanuc_m20ia_support/urdf/m20ia10l_macro.xacro (robot description, xacro)
@@ -109,5 +109,6 @@
       </collision>
     </link>
-    <link name="${prefix}tool0"/>
+    <link name="${prefix}flange" />
+    <link name="${prefix}tool0" />
     <!-- joints -->
     <joint name="${prefix}joint_1" type="revolute">
@@ -153,8 +154,13 @@
       <limit lower="-4.712389" upper="4.712389" effort="0" velocity="10.471980" />
     </joint>
-    <joint name="${prefix}joint_6-tool0" type="fixed">
+    <joint name="${prefix}joint_6-flange" type="fixed">
+      <origin xyz="0 0 0" rpy="0 0 0" />
+      <parent link="${prefix}link_6" />
+      <child link="${prefix}flange" />
+    </joint>
+    <joint name="${prefix}flange-tool0" type="fixed">
       <origin xyz="0 0 0" rpy="${pi} ${-pi/2.0} 0" />
-      <parent link="${prefix}link_6"/>
-      <child link="${prefix}tool0"/>
+      <parent link="${prefix}flange" />
+      <child link="${prefix}tool0" />
     </joint>
     <!-- ROS base_link to Fanuc World Coordinates transform -->

File: fanuc_m20ia_support/urdf/m20ia_macro.xacro (robot description, xacro)
@@ -109,5 +109,6 @@
       </collision>
     </link>
-    <link name="${prefix}tool0"/>
+    <link name="${prefix}flange" />
+    <link name="${prefix}tool0" />
     <!-- joints -->
     <joint name="${prefix}joint_1" type="revolute">
@@ -153,8 +154,13 @@
       <limit lower="-4.712389" upper="4.712389" effort="0" velocity="9.599311" />
     </joint>
-    <joint name="${prefix}joint_6-tool0" type="fixed">
+    <joint name="${prefix}joint_6-flange" type="fixed">
+      <origin xyz="0 0 0" rpy="0 0 0" />
+      <parent link="${prefix}link_6" />
+      <child link="${prefix}flange" />
+    </joint>
+    <joint name="${prefix}flange-tool0" type="fixed">
       <origin xyz="0 0 0" rpy="${pi} ${-pi/2.0} 0" />
-      <parent link="${prefix}link_6"/>
-      <child link="${prefix}tool0"/>
+      <parent link="${prefix}flange" />
+      <child link="${prefix}tool0" />
     </joint>
     <!-- ROS base_link to Fanuc World Coordinates transform -->

File: fanuc_m430ia_support/urdf/m430ia2f_macro.xacro (robot description, xacro)
@@ -94,5 +94,6 @@
       </collision>
     </link>
-    <link name="${prefix}tool0"/>
+    <link name="${prefix}flange" />
+    <link name="${prefix}tool0" />
     <!-- joints -->
     <joint name="${prefix}joint_1" type="revolute">
@@ -131,8 +132,13 @@
       <limit lower="-4.71" upper="4.71" effort="0" velocity="20.94"/>
     </joint>
-    <joint name="${prefix}joint_5-tool0" type="fixed">
+    <joint name="${prefix}joint_5-flange" type="fixed">
       <origin xyz="0 0 0" rpy="0 0 0" />
-      <parent link="${prefix}link_5"/>
-      <child link="${prefix}tool0"/>
+      <parent link="${prefix}link_5" />
+      <child link="${prefix}flange" />
+    </joint>
+    <joint name="${prefix}flange-tool0" type="fixed">
+      <origin xyz="0 0 0" rpy="0 0 0" />
+      <parent link="${prefix}flange" />
+      <child link="${prefix}tool0" />
     </joint>
     <!-- ROS base_link to Fanuc World Coordinates transform -->

File: fanuc_m430ia_support/urdf/m430ia2p_macro.xacro (robot description, xacro)
@@ -109,4 +109,5 @@
       </collision>
     </link>
+    <link name="${prefix}flange" />
     <link name="${prefix}tool0" />
     <!-- joints -->
@@ -153,7 +154,12 @@
       <limit lower="-4.71" upper="4.71" effort="0" velocity="12.57"/>
     </joint>
-    <joint name="${prefix}joint_6-tool0" type="fixed">
+    <joint name="${prefix}joint_6-flange" type="fixed">
       <origin xyz="0 0 0" rpy="0 0 0" />
       <parent link="${prefix}link_6" />
+      <child link="${prefix}flange" />
+    </joint>
+    <joint name="${prefix}flange-tool0" type="fixed">
+      <origin xyz="0 0 0" rpy="0 0 0" />
+      <parent link="${prefix}flange" />
       <child link="${prefix}tool0" />
     </joint>
